Commit message: Thesis 2026, Jurek Preisegger and Anton Espedalen

File: High_Level_Control_Computer/ap4_hlc_code/ap4hlc_ws/src/autonomous_platform_robot_description_pkg/src/description/imu.xacro (robot description, xacro)
@@ -21,5 +21,5 @@
         <parent link="base_link"/>
         <child link="imu_link"/>
-        <origin xyz="0 0 ${0.1+0.05+lidar_length/2.0}" rpy="0 0 0"/>
+        <origin xyz="0.5 0 ${0.1+0.05+lidar_length/2.0}" rpy="${pi} ${pi/2} 0"/>
     </joint>
     <gazebo reference="imu_link">

File: High_Level_Control_Computer/ap4_hlc_code/ap4hlc_ws/src/autonomous_platform_robot_description_pkg/src/description/lidar.xacro (robot description, xacro)
@@ -21,5 +21,5 @@
         <parent link="base_link"/>
         <child link="lidar_link"/>
-        <origin xyz="0.701 0 ${lidar_length/2.0}" rpy="0 0 0"/>
+        <origin xyz="0.721 0 ${lidar_length/2.0}" rpy="0 0 0"/>
     </joint>
     <gazebo reference="lidar_link">
